Commit message: urdf file updated

File: src/space_station_gnc/urdf/ISS_stationaryFromNasa.urdf (robot description, URDF)
Before this commit: robot ISS_stationaryFromNasa, 1 links, 0 joints
Links:
- link Root: geometry visual mesh filename=package://space_station_gnc/urdf/meshes/AMS2_000.obj scale=1. 1. 1.; visual mesh filename=package://space_station_gnc/urdf/meshes/Cube_001.obj scale=1. 1. 1.
