Commit message: space_station_gnc: Added thruster allocation matrix and reliable backend

File: space_station_gazebo/space_station_description/urdf/space_station.xacro (robot description, xacro)
@@ -4,4 +4,8 @@
 <xacro:include filename="$(find space_station_description)/urdf/space_station.trans" />
 <xacro:include filename="$(find space_station_description)/urdf/space_station.gazebo" />
+<xacro:property name="use_fixed_joint" value="true"/>
+<!-- <xacro:macro name="conditional_type" params="">
+  ${use_fixed_joint == 'true' ? 'fixed' : 'continuous'}
+</xacro:macro> -->
 <link name="base_link">
   <inertial>
@@ -604,5 +608,5 @@
   </collision>
 </link>
-<joint name="xp_th_1" type="continuous">
+<joint name="xp_th_1" type="${'fixed' if str(use_fixed_joint) == 'true' else 'continuous'}">
   <origin xyz="2.007871 -10.0 2.495824" rpy="0 0 0"/>
   <parent link="base_link"/>
@@ -610,5 +614,5 @@
   <axis xyz="0.0 1.0 0.0"/>
 </joint>
-<joint name="xp_th_2" type="continuous">
+<joint name="xp_th_2" type="${'fixed' if str(use_fixed_joint) == 'true' else 'continuous'}">
   <origin xyz="2.020507 -10.0 -2.503833" rpy="0 0 0"/>
   <parent link="base_link"/>
@@ -623,5 +627,5 @@
   <limit upper="0.0" lower="0.0" effort="100" velocity="100"/>
 </joint>
-<joint name="xp_th_3" type="continuous">
+<joint name="xp_th_3" type="${'fixed' if str(use_fixed_joint) == 'true' else 'continuous'}">
   <origin xyz="-1.984128 -9.9 2.498452" rpy="0 0 0"/>
   <parent link="base_link"/>
@@ -636,5 +640,5 @@
   <limit upper="0.0" lower="0.0" effort="100" velocity="100"/>
 </joint>
-<joint name="xp_th_4" type="continuous">
+<joint name="xp_th_4" type="${'fixed' if str(use_fixed_joint) == 'true' else 'continuous'}">
   <origin xyz="-1.991465 -10.0 -2.509155" rpy="0 0 0"/>
   <parent link="base_link"/>
@@ -642,5 +646,5 @@
   <axis xyz="0.0 1.0 0.0"/>
 </joint>
-<joint name="yn_th_1" type="continuous">
+<joint name="yn_th_1" type="${'fixed' if str(use_fixed_joint) == 'true' else 'continuous'}">
   <origin xyz="4.5 -9.0 0.0" rpy="0 0 0"/>
   <parent link="base_link"/>
@@ -648,5 +652,5 @@
   <axis xyz="1.0 0.0 0.0"/>
 </joint>
-<joint name="rsa_1" type="continuous">
+<joint name="rsa_1" type="${'fixed' if str(use_fixed_joint) == 'true' else 'continuous'}">
   <origin xyz="4.5 -6.0 0.0" rpy="0 0 0"/>
   <parent link="base_link"/>
@@ -654,5 +658,5 @@
   <axis xyz="1.0 0.0 0.0"/>
 </joint>
-<joint name="rsa_2" type="continuous">
+<joint name="rsa_2" type="${'fixed' if str(use_fixed_joint) == 'true' else 'continuous'}">
   <origin xyz="4.5 0.0 0.0" rpy="0 0 0"/>
   <parent link="base_link"/>
@@ -660,5 +664,5 @@
   <axis xyz="1.0 0.0 0.0"/>
 </joint>
-<joint name="rsa_3" type="continuous">
+<joint name="rsa_3" type="${'fixed' if str(use_fixed_joint) == 'true' else 'continuous'}">
   <origin xyz="4.5 6.0 0.0" rpy="0 0 0"/>
   <parent link="base_link"/>
@@ -666,5 +670,5 @@
   <axis xyz="1.0 0.0 0.0"/>
 </joint>
-<joint name="yn_th_2" type="continuous">
+<joint name="yn_th_2" type="${'fixed' if str(use_fixed_joint) == 'true' else 'continuous'}">
   <origin xyz="4.5 9.0 0.0" rpy="0 0 0"/>
   <parent link="base_link"/>
@@ -678,5 +682,5 @@
   <axis xyz="0.92388 0.0 0.382683"/>
 </joint>
-<joint name="zn_th_1" type="continuous">
+<joint name="zn_th_1" type="${'fixed' if str(use_fixed_joint) == 'true' else 'continuous'}">
   <origin xyz="-0.026882 -7.996277 4.4" rpy="0 0 0"/>
   <parent link="base_link"/>
@@ -684,5 +688,5 @@
   <axis xyz="0.0 0.0 -1.0"/>
 </joint>
-<joint name="zn_th_2" type="continuous">
+<joint name="zn_th_2" type="${'fixed' if str(use_fixed_joint) == 'true' else 'continuous'}">
   <origin xyz="0.0 8.0 4.4" rpy="0 0 0"/>
   <parent link="base_link"/>
@@ -697,5 +701,5 @@
   <limit upper="0.0" lower="0.0" effort="100" velocity="100"/>
 </joint>
-<joint name="yp_th_1" type="continuous">
+<joint name="yp_th_1" type="${'fixed' if str(use_fixed_joint) == 'true' else 'continuous'}">
   <origin xyz="-4.5 -9.0 0.0" rpy="0 0 0"/>
   <parent link="base_link"/>
@@ -703,5 +707,5 @@
   <axis xyz="-1.0 0.0 0.0"/>
 </joint>
-<joint name="lsa_1" type="continuous">
+<joint name="lsa_1" type="${'fixed' if str(use_fixed_joint) == 'true' else 'continuous'}">
   <origin xyz="-4.5 -6.0 0.0" rpy="0 0 0"/>
   <parent link="base_link"/>
@@ -716,5 +720,5 @@
   <limit upper="0.0" lower="0.0" effort="100" velocity="100"/>
 </joint>
-<joint name="lsa_2" type="continuous">
+<joint name="lsa_2" type="${'fixed' if str(use_fixed_joint) == 'true' else 'continuous'}">
   <origin xyz="-4.5 0.0 0.0" rpy="0 0 0"/>
   <parent link="base_link"/>
@@ -722,5 +726,5 @@
   <axis xyz="-1.0 0.0 0.0"/>
 </joint>
-<joint name="yp_th_2" type="continuous">
+<joint name="yp_th_2" type="${'fixed' if str(use_fixed_joint) == 'true' else 'continuous'}">
   <origin xyz="-4.5 9.0 0.0" rpy="0 0 0"/>
   <parent link="base_link"/>
@@ -728,5 +732,5 @@
   <axis xyz="-1.0 0.0 0.0"/>
 </joint>
-<joint name="lsa_3" type="continuous">
+<joint name="lsa_3" type="${'fixed' if str(use_fixed_joint) == 'true' else 'continuous'}">
   <origin xyz="-4.5 6.0 0.0" rpy="0 0 0"/>
   <parent link="base_link"/>
@@ -734,5 +738,5 @@
   <axis xyz="-1.0 0.0 0.0"/>
 </joint>
-<joint name="zp_th_1" type="continuous">
+<joint name="zp_th_1" type="${'fixed' if str(use_fixed_joint) == 'true' else 'continuous'}">
   <origin xyz="0.00669 -7.997906 -4.4" rpy="0 0 0"/>
   <parent link="base_link"/>
@@ -740,5 +744,5 @@
   <axis xyz="0.0 0.0 1.0"/>
 </joint>
-<joint name="zp_th_2" type="continuous">
+<joint name="zp_th_2" type="${'fixed' if str(use_fixed_joint) == 'true' else 'continuous'}">
   <origin xyz="0.001241 8.003055 -4.4" rpy="0 0 0"/>
   <parent link="base_link"/>
@@ -746,5 +750,5 @@
   <axis xyz="0.0 0.0 1.0"/>
 </joint>
-<joint name="xn_th_1" type="continuous">
+<joint name="xn_th_1" type="${'fixed' if str(use_fixed_joint) == 'true' else 'continuous'}">
   <origin xyz="-2.0 10.0 2.5" rpy="0 0 0"/>
   <parent link="base_link"/>
@@ -752,5 +756,5 @@
   <axis xyz="0.0 -1.0 0.0"/>
 </joint>
-<joint name="xn_th_2" type="continuous">
+<joint name="xn_th_2" type="${'fixed' if str(use_fixed_joint) == 'true' else 'continuous'}">
   <origin xyz="-1.982378 10.0 -2.506934" rpy="0 0 0"/>
   <parent link="base_link"/>
@@ -758,5 +762,5 @@
   <axis xyz="0.0 -1.0 0.0"/>
 </joint>
-<joint name="xn_th_3" type="continuous">
+<joint name="xn_th_3" type="${'fixed' if str(use_fixed_joint) == 'true' else 'continuous'}">
   <origin xyz="2.000104 10.0 -2.503617" rpy="0 0 0"/>
   <parent link="base_link"/>
@@ -770,5 +774,5 @@
   <axis xyz="0.0 1.0 0.0"/>
 </joint>
-<joint name="xn_th_4" type="continuous">
+<joint name="xn_th_4" type="${'fixed' if str(use_fixed_joint) == 'true' else 'continuous'}">
   <origin xyz="2.0 10.0 2.5" rpy="0 0 0"/>
   <parent link="base_link"/>
